Commit message: updated urdf, fixed joint4, implemented FK,IK. TODO: fix gazebo and traj issues

File: urdf/robot_old.urdf.xacro (robot description, xacro)
@@ -13,12 +13,12 @@
         rpy="0 0 0" />
       <mass
-        value="400" />
-      <inertia
-        ixx="10"
-        ixy="10"
-        ixz="10"
-        iyy="10"
-        iyz="10"
-        izz="10" />
+        value="61.0676487684592" /> #TODO
+      <inertia
+        ixx="0.000760494487568691"
+        ixy="7.86857711947688E-08"
+        ixz="3.40719385268755E-07"
+        iyy="0.00077439103050546"
+        iyz="-3.4527228052956E-06"
+        izz="0.00100204247644816" />
     </inertial>
     <visual>
@@ -59,12 +59,12 @@
         rpy="0 0 0" />
       <mass
-        value="40" />
-      <inertia
-        ixx="31.7856467096501"
-        ixy="0.000533354169263688"
-        ixz="-0.00809623107461862"
-        iyy="31.7878803195643"
-        iyz="0.0058154121088785"
-        izz="31.7408712499535" />
+        value="2.0" />
+      <inertia
+        ixx="0.00120409888419921"
+        ixy="-1.39536489001303E-07"
+        ixz="4.27140501519446E-08"
+        iyy="0.00111869817012112"
+        iyz="0.000101273303403283"
+        izz="0.000911594560955689" />
     </inertial>
     <visual>
@@ -117,12 +117,12 @@
         rpy="0 0 0" />
       <mass
-        value="40" />
-      <inertia
-        ixx="31.7856467096501"
-        ixy="0.000533354169263688"
-        ixz="-0.00809623107461862"
-        iyy="31.7878803195643"
-        iyz="0.0058154121088785"
-        izz="31.7408712499535" />
+        value="3.42" />
+      <inertia
+        ixx="0.019297803356077"
+        ixy="-1.47617988019155E-07"
+        ixz="7.37970525209698E-08"
+        iyy="0.00210354731087032"
+        iyz="-0.00135595921273946"
+        izz="0.0187229765717406" />
     </inertial>
     <visual>
@@ -175,12 +175,12 @@
         rpy="0 0 0" />
       <mass
-        value="40" />
-      <inertia
-        ixx="31.7856467096501"
-        ixy="0.000533354169263688"
-        ixz="-0.00809623107461862"
-        iyy="31.7878803195643"
-        iyz="0.0058154121088785"
-        izz="31.7408712499535" />
+        value="1.26" />
+      <inertia
+        ixx="0.000638857905152697"
+        ixy="4.44620386081057E-08"
+        ixz="0.00056680409821328"
+        iyy="0.00701668679175095"
+        iyz="-3.10409752224366E-10"
+        izz="0.00683638640718249" />
     </inertial>
     <visual>
@@ -233,12 +233,12 @@
         rpy="0 0 0" />
       <mass
-        value="40" />
-      <inertia
-        ixx="31.7856467096501"
-        ixy="0.000533354169263688"
-        ixz="-0.00809623107461862"
-        iyy="31.7878803195643"
-        iyz="0.0058154121088785"
-        izz="31.7408712499535" />
+        value="0.8" />
+      <inertia
+        ixx="0.000178924033269713"
+        ixy="6.66496087009546E-10"
+        ixz="-1.68870620715207E-05"
+        iyy="0.000215917794765493"
+        iyz="-8.81135271781819E-10"
+        izz="0.000181683883551313" />
     </inertial>
     <visual>
@@ -291,12 +291,12 @@
         rpy="0 0 0" />
       <mass
-        value="40" />
-      <inertia
-        ixx="31.7856467096501"
-        ixy="0.000533354169263688"
-        ixz="-0.00809623107461862"
-        iyy="31.7878803195643"
-        iyz="0.0058154121088785"
-        izz="31.7408712499535" />
+        value="0.8" />
+      <inertia
+        ixx="0.00021591792388467"
+        ixy="7.65171892824432E-10"
+        ixz="8.23290393884545E-10"
+        iyy="0.00017892418948679"
+        iyz="1.68871139435162E-05"
+        izz="0.000181684105968982" />
     </inertial>
     <visual>
@@ -349,12 +349,12 @@
         rpy="0 0 0" />
       <mass
-        value="40" />
-      <inertia
-        ixx="31.7856467096501"
-        ixy="0.000533354169263688"
-        ixz="-0.00809623107461862"
-        iyy="31.7878803195643"
-        iyz="0.0058154121088785"
-        izz="31.7408712499535" />
+        value="0.35" />
+      <inertia
+        ixx="0.00333846848595568"
+        ixy="1.88415933556498E-12"
+        ixz="-7.36290023764471E-12"
+        iyy="0.00333887923474237"
+        iyz="-5.32112866368567E-07"
+        izz="0.00032876963440072" />
     </inertial>
     <visual>
@@ -407,12 +407,12 @@
         rpy="0 0 0" />
       <mass
-        value="1" />
-      <inertia
-        ixx="31.7856467096501"
-        ixy="0.000533354169263688"
-        ixz="-0.00809623107461862"
-        iyy="31.7878803195643"
-        iyz="0.0058154121088785"
-        izz="31.7408712499535" />
+        value="0.0908764844935512" />
+      <inertia
+        ixx="0.000450562904874952"
+        ixy="1.71281909805966E-20"
+        ixz="2.77793826384743E-18"
+        iyy="0.0004503722428556"
+        iyz="9.96040593377829E-07"
+        izz="1.26158531179263E-05" />
     </inertial>
     <visual>
@@ -465,12 +465,12 @@
         rpy="0 0 0" />
       <mass
-        value="0.5" />
-      <inertia
-        ixx="31.7856467096501"
-        ixy="0.000533354169263688"
-        ixz="-0.00809623107461862"
-        iyy="31.7878803195643"
-        iyz="0.0058154121088785"
-        izz="31.7408712499535" />
+        value="0.449460569532232" />
+      <inertia
+        ixx="0.00185160492644654"
+        ixy="5.78351491181251E-07"
+        ixz="8.73825554656471E-07"
+        iyy="0.00141795601961042"
+        iyz="-0.000685950601972587"
+        izz="0.000615251613020217" />
     </inertial>
     <visual>
