Commit message: added teleop, updated urdf TODO: fix Joint 4

File: urdf/charging_robot.urdf.xacro (robot description, xacro)
@@ -12,5 +12,5 @@
         rpy="0 0 0" />
       <mass
-        value="0.610676487684592" />
+        value="6.10676487684592" /> #"0.610676487684592""
       <inertia
         ixx="0.000760494487568691"
@@ -99,5 +99,5 @@
   <joint
     name="Joint1"
-    type="continuous">
+    type="revolute">
     <origin
       xyz="0 0 0.0844"
@@ -109,7 +109,7 @@
     <axis
       xyz="0 1 0" />
-    <limit
-      lower="0"
-      upper="0"
+     <limit
+      lower="-3.1415"
+      upper="3.1415"
       effort="0"
       velocity="0" />
@@ -157,5 +157,5 @@
   <joint
     name="Joint2"
-    type="continuous">
+    type="revolute">
     <origin
       xyz="0 0.056958 0.17256"
@@ -167,4 +167,9 @@
     <axis
       xyz="0 0 -1" /> #0 0.087156 -0.99619
+    <limit
+      lower="-3.1415"
+      upper="3.1415"
+      effort="0"
+      velocity="0" />
   </joint>
   <link
@@ -210,5 +215,5 @@
   <joint
     name="Joint3"
-    type="continuous">
+    type="revolute">
     <origin
       xyz="0 -0.45207 -0.23019"
@@ -219,5 +224,10 @@
       link="Link3" />
     <axis
-      xyz="0 0 -1" /> # 0.087156 0 -0.99619
+      xyz="0 0 1" /> # 0.087156 0 -0.99619
+    <limit
+      lower="-3.1415"
+      upper="3.1415"
+      effort="0"
+      velocity="0" />
   </joint>
   <link
@@ -263,5 +273,5 @@
   <joint
     name="Joint4"
-    type="continuous"> #Changed to continuous
+    type="revolute"> #Changed to revolute
     <origin
       xyz="0.0078715 0 -0.12719"
@@ -272,5 +282,10 @@
       link="Link4" />
     <axis
-      xyz="0 0 0" />
+      xyz="1 0 0 " />
+    <limit
+      lower="-3.1415"
+      upper="3.1415"
+      effort="0"
+      velocity="0" />
   </joint>
   <link
@@ -327,6 +342,6 @@
       xyz="1 0 0" />
     <limit
-      lower="0"
-      upper="0"
+      lower="-3.1415"
+      upper="3.1415"
       effort="0"
       velocity="0" />
@@ -374,5 +389,5 @@
   <joint
     name="Joint6"
-    type="continuous">
+    type="revolute">
     <origin
       xyz="0 -0.2924 0"
@@ -384,4 +399,9 @@
     <axis
       xyz="0 0 1" />
+    <limit
+      lower="-3.1415"
+      upper="3.1415"
+      effort="0"
+      velocity="0" />
   </joint>
   <link
@@ -439,5 +459,5 @@
     <limit
       lower="0"
-      upper="0"
+      upper="0.2"
       effort="0"
       velocity="0" />

Commit message: fixed few errors

File: urdf/charging_robot.urdf.xacro (robot description, xacro)
@@ -13,12 +13,12 @@
         rpy="0 0 0" />
       <mass
-        value="400" />
-      <inertia
-        ixx="10"
-        ixy="10"
-        ixz="10"
-        iyy="10"
-        iyz="10"
-        izz="10" />
+        value="40000" />
+      <inertia
+        ixx="1000"
+        ixy="1000"
+        ixz="1000"
+        iyy="1000"
+        iyz="1000"
+        izz="1000" />
     </inertial>
     <visual>
